File: power_source/power_source.kicad_pcb (KiCad board)
At the start: 2 copper layers, 21 parts, among them J1 Traf secondary, J2 Traf Primary, J3 Input 230V AC, J4 Power, J5 5V DC, J6 12V DC, K1 SANYOU_SRD_Form_C, K2 SANYOU_SRD_Form_C, K3 SANYOU_SRD_Form_C, Q1 BC337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

Commit message: Wip
Parts:
- added C1: 100nF, Capacitor_THT:C_Disc_D10.0mm_W2.5mm_P5.00mm, F.Cu at (45.0, 137.5)
- added C2: 100nF, Capacitor_THT:C_Disc_D10.0mm_W2.5mm_P5.00mm, F.Cu at (130.0, 132.5)
- added C3: 2200uF, Capacitor_THT:CP_Radial_D18.0mm_P7.50mm, F.Cu at (60.0, 135.0)
- added C4: 2200uF, Capacitor_THT:CP_Radial_D18.0mm_P7.50mm, F.Cu at (115.0, 135.0)
- added D4: B40C1500G, Diode_THT:Diode_Bridge_Round_D9.8mm, F.Cu at (32.0, 137.5)
- added J7: Input 12V AC, Connector_Wire:SolderWire-0.5sqmm_1x02_P4.8mm_D0.9mm_OD2.3mm, F.Cu at (22.5, 137.5)
- added J8: Power amplifier output, Connector_Wire:SolderWire-0.5sqmm_1x04_P4.8mm_D0.9mm_OD2.3mm, F.Cu at (60.6, 42.5)
- added J9: Speakers, Connector_Wire:SolderWire-0.5sqmm_1x04_P4.8mm_D0.9mm_OD2.3mm, F.Cu at (125.5, 42.4)
- added U2: LM7812_TO220, Package_TO_SOT_THT:TO-220-3_Vertical, F.Cu at (87.5, 134.9)
- J1: footprint Connector_Wire:SolderWire-0.5sqmm_1x04_P4.6mm_D0.9mm_OD2.1mm -> Connector_Wire:SolderWire-0.5sqmm_1x04_P4.8mm_D0.9mm_OD2.3mm
- J2: footprint Connector_Wire:SolderWire-0.5sqmm_1x02_P4.6mm_D0.9mm_OD2.1mm -> Connector_Wire:SolderWire-0.75sqmm_1x02_P4.8mm_D1.25mm_OD2.3mm
- J3: footprint Connector_Wire:SolderWire-0.5sqmm_1x02_P4.6mm_D0.9mm_OD2.1mm -> Connector_Wire:SolderWire-0.5sqmm_1x02_P4.8mm_D0.9mm_OD2.3mm
- J4: value Power -> Power Amplifier Power
- J5, J6: footprint Connector_Wire:SolderWire-0.5sqmm_1x02_P4.6mm_D0.9mm_OD2.1mm -> Connector_JST:JST_XH_B2B-XH-A_1x02_P2.50mm_Vertical
- PS2: value HLK-PM12 -> HLK-PM01
- moved J1 165.4 mm to (22.5, 60.6), turned to -90 degrees
- moved J4 153.1 mm to (40.4, 42.5)
- moved K1 145.3 mm to (36.5, 67.5)
- moved J3 101.3 mm to (22.5, 112.7), turned to -90 degrees
- moved J2 100.0 mm to (22.5, 87.7), turned to -90 degrees
- moved Q1 96.4 mm to (67.5, 68.5), turned to 90 degrees
- moved R1 93.4 mm to (72.5, 72.7), turned to 90 degrees
- moved D1 92.3 mm to (60.0, 72.7), turned to 90 degrees
- moved R2 85.5 mm to (116.0, 117.5)
- moved U1 83.2 mm to (98.9, 118.6), turned to 180 degrees
- moved PS1 73.6 mm to (33.0, 112.5)
- moved R3 73.3 mm to (136.0, 117.5)
- moved K2 66.3 mm to (120.0, 98.5), turned to 90 degrees
- moved D2 62.9 mm to (126.0, 104.0), turned to 180 degrees
- moved D3 55.3 mm to (146.2, 104.0), turned to 180 degrees
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Connections:
- J2 pad 1: unconnected-(J2-Pin_1-Pad1) -> Traf in
- J2 pad 2: unconnected-(J2-Pin_2-Pad2) -> 220V AC N
- J3 pad 1: Net-(J3-Pin_1) -> 220V AC R
- J3 pad 2: Net-(J3-Pin_2) -> 220V AC N
- J5 pad 1: unconnected-(J5-Pin_1-Pad1) -> Net-(J5-Pin_1)
- J5 pad 2: GND -> Net-(J5-Pin_2)
- J6 pad 1: unconnected-(J6-Pin_1-Pad1) -> Net-(D4--)
- J6 pad 2: GND -> Net-(J6-Pin_2)
- K1 pad 1: unconnected-(K1-Pad1) -> 220V AC R
- K1 pad 3: unconnected-(K1-Pad3) -> Traf in
- K2 pad 1: unconnected-(K2-Pad1) -> IN LSP+
- K2 pad 3: unconnected-(K2-Pad3) -> OUT LSP+
- K3 pad 1: unconnected-(K3-Pad1) -> IN RSP+
- K3 pad 3: unconnected-(K3-Pad3) -> OUT RSP+
- PS1 pad 1: Net-(J3-Pin_1) -> 220V AC R
- PS1 pad 2: Net-(J3-Pin_2) -> 220V AC N
- PS1 pad 3: GND -> Net-(J5-Pin_1)
- PS1 pad 4: +5V -> Net-(J5-Pin_2)
- PS2 pad 1: Net-(J3-Pin_1) -> 220V AC N
- PS2 pad 2: Net-(J3-Pin_2) -> 220V AC R
- PS2 pad 4: +12V -> +5V
- U1 pad 1: GND -> +5V
- U1 pad 10: REL2 -> REL1
- U1 pad 12: GND -> +5V
- U1 pad 13: +5V -> 5V
- U1 pad 14: +5V -> 5V
- U1 pad 15: GND -> +5V
- U1 pad 16: GND -> +5V
- U1 pad 19: GND -> +5V
- U1 pad 24: GND -> +5V
- U1 pad 27: GND -> +5V
- U1 pad 30: GND -> +5V
- U1 pad 4: REL3 -> REL2
- U1 pad 6: GND -> +5V
- U1 pad 8: GND -> +5V
- U1 pad 9: REL1 -> REL3
Routing:
- net +5V: track 0.00 -> 185.1 mm
- net Net-(J5-Pin_1): track 0.00 -> 127.3 mm
- net Net-(D4--): track 0.00 -> 117.7 mm
- net Net-(J5-Pin_2): track 0.00 -> 110.9 mm
- net IN RSP+: track 0.00 -> 102.3 mm
- net IN LSP+: track 0.00 -> 96.6 mm
- net 220V AC R: track 0.00 -> 82.0 mm
- net Net-(J8-Pin_4): track 0.00 -> 81.0 mm, vias 0 -> 2
- net Net-(J8-Pin_2): track 0.00 -> 75.4 mm, vias 0 -> 4
- net Net-(J6-Pin_2): track 0.00 -> 60.6 mm
- net Net-(D4-+): track 0.00 -> 60.2 mm
- net 220V AC N: track 0.00 -> 59.2 mm
- net OUT RSP+: track 0.00 -> 47.6 mm
- net REL3: track 0.00 -> 47.0 mm, vias 0 -> 2
- net Net-(J1-Pin_4): track 0.00 -> 43.9 mm
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- added copper zone on B.Cu, net GND
Other:
- board outline added: 137.5 x 112.5 mm

Commit message: WIP
Parts:
- removed J9: Speakers, Connector_Wire:SolderWire-0.5sqmm_1x04_P4.8mm_D0.9mm_OD2.3mm
- added J10: Trafo, TerminalBlock:TerminalBlock_Altech_AK300-4_P5.00mm, F.Cu at (22.5, 60.0)
- J1: value Traf secondary -> Power Ampli Power; footprint Connector_Wire:SolderWire-0.5sqmm_1x04_P4.8mm_D0.9mm_OD2.3mm -> TerminalBlock:TerminalBlock_Altech_AK300-3_P5.00mm
- J4: value Power Amplifier Power -> Power Ampl output; footprint Connector_Wire:SolderWire-0.5sqmm_1x03_P4.8mm_D0.9mm_OD2.3mm -> TerminalBlock:TerminalBlock_Altech_AK300-4_P5.00mm
- J8: value Power amplifier output -> Speakers; footprint Connector_Wire:SolderWire-0.5sqmm_1x04_P4.8mm_D0.9mm_OD2.3mm -> TerminalBlock:TerminalBlock_Altech_AK300-4_P5.00mm
- moved J8 64.4 mm to (125.0, 42.5)
- moved J1 25.0 mm to (39.7, 42.5), turned to 0 degrees
- moved J4 19.6 mm to (60.0, 42.5)
- moved J7 10.0 mm to (22.5, 127.5)
- moved J5 7.50 mm to (137.5, 145.0)
- moved J6 7.50 mm to (125.0, 145.0)
- moved C4 5.59 mm to (110.0, 137.5)
Connections:
- J1 pad 3: Net-(J1-Pin_2) -> Net-(J1-Pin_3)
- J4 pad 1: Net-(J1-Pin_1) -> IN LSP+
- J4 pad 2: Net-(J1-Pin_2) -> Net-(J4-Pin_2)
- J4 pad 3: Net-(J1-Pin_4) -> IN RSP+
- J8 pad 1: IN LSP+ -> OUT LSP+
- J8 pad 2: Net-(J8-Pin_2) -> Net-(J4-Pin_2)
- J8 pad 3: IN RSP+ -> OUT RSP+
- J8 pad 4: Net-(J8-Pin_4) -> Net-(J4-Pin_4)
Routing:
- net Net-(J8-Pin_4): track 81.0 -> 0.00 mm, vias 2 -> 0
- net Net-(J4-Pin_4): track 0.00 -> 81.0 mm, vias 0 -> 2
- net Net-(J8-Pin_2): track 75.4 -> 0.00 mm, vias 4 -> 0
- net Net-(J4-Pin_2): track 0.00 -> 74.8 mm, vias 0 -> 4
- net Net-(J1-Pin_3): track 0.00 -> 44.0 mm
- net Net-(J1-Pin_4): track 43.9 -> 0.00 mm
- net Net-(D4--): track 117.7 -> 128.3 mm
- net Net-(J7-Pin_1): track 16.9 -> 25.5 mm
- net Net-(J6-Pin_2): track 60.6 -> 52.7 mm
- net Net-(J7-Pin_2): track 9.57 -> 17.1 mm
- net Net-(J5-Pin_2): track 110.9 -> 106.4 mm
- net Net-(J5-Pin_1): track 127.3 -> 122.7 mm
- net OUT LSP+: track 42.1 -> 42.9 mm
- net Net-(J1-Pin_1): track 26.6 -> 26.1 mm
Other:
- outline, holes or cut-outs redrawn
