File: delay_circuit/delay_circuit.kicad_sch (KiCad schematic)
At the start: 26 parts, among them J1 IN 12V AC, J2 OUT 230V AC, J3 IN 230V AC, J4 From Trfo Output, J5 OUT 5V CC, J6 To Power Ampli Power IN, J7 From Ampli Output, J8 OUT 12V CC, J9 To Speakers, K1 SANYOU_SRD_Form_C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

Commit message: WIP
Parts:
- Q2: footprint Package_TO_SOT_THT:TO-3P-3_Vertical -> Package_TO_SOT_THT:TO-126-3_Vertical
Changed lines of the file:
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@@
 			)
 		)
-		(property "Footprint" "Package_TO_SOT_THT:TO-3P-3_Vertical"
+		(property "Footprint" "Package_TO_SOT_THT:TO-126-3_Vertical"
 			(at 172.72 109.22 0)
 			(effects

Commit message: Improved board.
Parts:
- PS1, PS2: footprint Converter_ACDC:Converter_ACDC_Hi-Link_HLK-PMxx -> Components:Converter_ACDC_Hi-Link_HLK-PMxx
- Q2: footprint Package_TO_SOT_THT:TO-126-3_Vertical -> Components:TO-126-3_Vertical
- R1, R2, R3: footprint Resistor_THT:R_Axial_DIN0411_L9.9mm_D3.6mm_P15.24mm_Horizontal -> Resistor_THT:R_Axial_DIN0207_L6.3mm_D2.5mm_P15.24mm_Horizontal
Connections:
- net IN SP L+: now also K1.3; no longer K1.4
- net IN SP R+: now also K2.3; no longer K2.4
Changed lines of the file:
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@@
-		)
-	)
-	(global_label "IN SP R+"
-		(shape input)
-		(at 170.18 78.74 0)
-		(fields_autoplaced yes)
-		(effects
-			(font
-				(size 1.27 1.27)
-			)
-			(justify left)
-		)
-		(property "Intersheetrefs" "${INTERSHEET_REFS}"
-			(at 182.3576 78.74 0)
-			(effects
-				(font
-					(size 1.27 1.27)
-				)
-				(justify left)
-				(hide yes)
-			)
 		)
 	)
@@
 		)
 	)
-	(global_label "IN SP L+"
+	(global_label "IN SP R+"
 		(shape input)
-		(at 128.27 78.74 0)
+		(at 170.18 83.82 0)
 		(fields_autoplaced yes)
 		(effects
@@
 		)
 		(property "Intersheetrefs" "${INTERSHEET_REFS}"
-			(at 140.2057 78.74 0)
+			(at 182.3576 83.82 0)
+			(effects
+				(font
+					(size 1.27 1.27)
+				)
+				(justify left)
+				(hide yes)
+			)
+		)
+	)
+	(global_label "IN SP L+"
+		(shape input)
+		(at 128.27 83.82 0)
+		(fields_autoplaced yes)
+		(effects
+			(font
+				(size 1.27 1.27)
+			)
+			(justify left)
+		)
+		(property "Intersheetrefs" "${INTERSHEET_REFS}"
+			(at 140.2057 83.82 0)
 			(effects
 				(font
@@
 			)
 		)
-		(property "Footprint" "Package_TO_SOT_THT:TO-126-3_Vertical"
+		(property "Footprint" "Components:TO-126-3_Vertical"
 			(at 172.72 109.22 0)
 			(effects
@@
 			)
 		)
-		(property "Footprint" "Resistor_THT:R_Axial_DIN0411_L9.9mm_D3.6mm_P15.24mm_Horizontal"
+		(property "Footprint" "Resistor_THT:R_Axial_DIN0207_L6.3mm_D2.5mm_P15.24mm_Horizontal"
 			(at 78.232 93.98 90)
 			(effects
@@
 			)
 		)
-		(property "Footprint" "Converter_ACDC:Converter_ACDC_Hi-Link_HLK-PMxx"
+		(property "Footprint" "Components:Converter_ACDC_Hi-Link_HLK-PMxx"
 			(at 53.34 99.06 0)
 			(effects
@@
 			)
 		)
-		(property "Footprint" "Resistor_THT:R_Axial_DIN0411_L9.9mm_D3.6mm_P15.24mm_Horizontal"
+		(property "Footprint" "Resistor_THT:R_Axial_DIN0207_L6.3mm_D2.5mm_P15.24mm_Horizontal"
 			(at 87.63 105.918 90)
 			(effects
@@
 			)
 		)
-		(property "Footprint" "Converter_ACDC:Converter_ACDC_Hi-Link_HLK-PMxx"
+		(property "Footprint" "Components:Converter_ACDC_Hi-Link_HLK-PMxx"
 			(at 53.34 118.11 0)
 			(effects
@@
 			)
 		)
-		(property "Footprint" "Resistor_THT:R_Axial_DIN0411_L9.9mm_D3.6mm_P15.24mm_Horizontal"
+		(property "Footprint" "Resistor_THT:R_Axial_DIN0207_L6.3mm_D2.5mm_P15.24mm_Horizontal"
 			(at 98.552 114.3 90)
 			(effects

Commit message: Reduced board size.
Connections:
- net at J5.1 (Pin_1): now also PS2.3 (-Vout); no longer PS2.4 (+Vout)
- net at J5.2 (Pin_2): now also PS2.4 (+Vout); no longer PS2.3 (-Vout)
Other:
- moved on the sheet: J5
Changed lines of the file:
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@@
 	(symbol
 		(lib_id "Connector:Conn_01x02_Pin")
-		(at 68.58 107.95 0)
-		(mirror y)
+		(at 68.58 110.49 180)
 		(unit 1)
 		(exclude_from_sim no)
@@
 		(dnp no)
 		(property "Reference" "J5"
-			(at 66.294 105.156 0)
+			(at 66.294 113.284 0)
 			(effects
 				(font
@@
 		)
 		(property "Value" "OUT 5V CC"
-			(at 66.294 113.792 0)
+			(at 66.294 104.648 0)
 			(effects
 				(font
@@
 		)
 		(property "Footprint" "Connector_JST:JST_XH_B2B-XH-A_1x02_P2.50mm_Vertical"
-			(at 68.58 107.95 0)
+			(at 68.58 110.49 0)
 			(effects
 				(font
@@
 		)
 		(property "Datasheet" "~"
-			(at 68.58 107.95 0)
+			(at 68.58 110.49 0)
 			(effects
 				(font
@@
 		)
 		(property "Description" "Generic connector, single row, 01x02, script generated"
-			(at 68.58 107.95 0)
+			(at 68.58 110.49 0)
 			(effects
 				(font
@@
 		)
 		(instances
-			(project ""
+			(project "delay_circuit"
 				(path "/6cfd9bb4-f1a0-4251-8e2c-45a42268d192"
 					(reference "J5")
