File: power_board/power_board.kicad_sch (KiCad schematic)
At the start: 26 parts, among them J1 From Trfo Output, J2 IN 12V AC, J3 OUT 230V AC, J4 IN 230V AC, J5 To Power Ampli Power IN, J6 OUT 5V CC, J7 From Ampli Output, J8 To Speakers, J9 OUT 12V CC, K1 SANYOU_SRD_Form_C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

Commit message: Power board.
Parts:
- Q1: value NPN -> BC171
- Q2: value NPN -> BD235
Connections:
- net 230VAC: now reaches J3.1 (Pin_1), J4.1 (Pin_1), PS1.1 (AC/L), PS2.1 (AC/L)
- net 230V AC (N): now reaches J3.2 (Pin_2), J4.2 (Pin_2), PS1.2 (AC/N), PS2.2 (AC/N)
- net SP L-: now reaches J7.2 (Pin_2), J8.3 (Pin_3)
- net SP R-: now reaches J7.4 (Pin_4), J8.1 (Pin_1)
- net 5V Gnd: now reaches J6.1 (Pin_1), PS2.3 (-Vout)
- net +5V: now reaches J6.2 (Pin_2), PS2.4 (+Vout)
- net +12V: now reaches C4.1, C5.1, J9.2 (Pin_2), U1.3 (VO)
- net L1 +: now reaches J1.1 (Pin_1), J5.3 (Pin_3)
- net Power GND: now reaches J1.2 (Pin_2), J1.3 (Pin_3), J5.2 (Pin_2)
- net L2 -: now reaches J1.4 (Pin_4), J5.1 (Pin_1)
Other:
- moved on the sheet: J5, J6, J7, J8
