File: power_board/power_board.kicad_pcb (KiCad board)
At the start: 2 copper layers, 83 x 111.5 mm, 26 parts, among them J1 From Trfo Output, J2 IN 12V AC, J3 OUT 230V AC, J4 IN 230V AC, J5 To Power Ampli Power IN, J6 OUT 5V CC, J7 From Ampli Output, J8 To Speakers, J9 OUT 12V CC, K1 SANYOU_SRD_Form_C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

Commit message: Power board.
Parts:
- Q1: value NPN -> BC171
- Q2: value NPN -> BD235
- moved R1 29.9 mm to (100.5, 91.3)
- moved R2 25.7 mm to (95.0, 106.5), turned to 90 degrees
- moved C3 12.9 mm to (98.2, 111.4), turned to 180 degrees
- moved J6 8.51 mm to (102.5, 126.0)
- moved Q1 8.32 mm to (96.0, 85.9)
- moved J9 7.27 mm to (92.2, 126.0)
- moved J8 7.11 mm to (99.0, 49.5)
- moved Q2 6.16 mm to (98.3, 79.5), turned to 180 degrees
- moved C2 6.02 mm to (40.5, 126.0)
- moved J1 6.01 mm to (42.0, 35.5)
- moved C4 6.00 mm to (81.0, 127.5)
- moved C5 6.00 mm to (54.5, 126.5)
- moved J2 6.00 mm to (42.0, 58.7)
- moved J3 6.00 mm to (42.0, 72.7)
- moved J4 6.00 mm to (42.0, 86.2)
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Connections:
- net Net-(J1-Pin_1) renamed L1 +
- net Net-(J1-Pin_2) renamed Power GND
- net Net-(J1-Pin_4) renamed L2 -
- net Net-(J3-Pin_1) renamed 230VAC
- net Net-(J3-Pin_2) renamed 230V AC (N)
- net Net-(J6-Pin_1) renamed 5V Gnd
- net Net-(J6-Pin_2) renamed +5V
- net Net-(J7-Pin_2) renamed SP L-
- net Net-(J7-Pin_4) renamed SP R-
- net Net-(J9-Pin_2) renamed +12V
Routing:
- net Net-(D2-A): track 74.6 -> 117.4 mm
- net Net-(D2-K): track 77.7 -> 100.7 mm
- net 12V GND: track 106.7 -> 124.5 mm
- net Net-(C3-Pad1): track 25.8 -> 10.5 mm
- net 230V AC (N): track 76.0 -> 67.8 mm
- net L1 +: track 18.9 -> 12.8 mm
- net +5V: track 15.8 -> 21.9 mm
- net Net-(Q1-E): track 19.1 -> 13.7 mm
- net 230VAC: track 62.8 -> 57.8 mm
- net Power GND: track 29.8 -> 25.2 mm
- net 5V Gnd: track 31.8 -> 35.9 mm
- net L2 -: track 33.3 -> 29.4 mm
- net 0: track 64.9 -> 68.6 mm
- net +12V: track 57.9 -> 61.2 mm
- net Net-(J2-Pin_1): track 91.0 -> 94.2 mm
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Other:
- board size 83 x 111.5 mm -> 73 x 109.5 mm
- board text added: "+"
- board text added: "-"
- board text added: "12 Vcc"
- board text added: "5 Vcc"

Commit message: Power board.
Routing:
- net 230VAC: track 57.8 -> 61.4 mm
Changed lines of the file:
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@@
 		)
 		(property "Value" "IN 230V AC"
-			(at 2.78 7.75 90)
+			(at 2.78 7 90)
 			(layer "F.Fab")
 			(effects
@@
 		)
 		(property "Value" "IN 12V AC"
-			(at 2.78 7.75 90)
+			(at 2.78 7 90)
 			(layer "F.Fab")
 			(effects
@@
 		)
 		(property "Value" "OUT 230V AC"
-			(at 2.78 7.75 90)
+			(at 2.78 7 90)
 			(layer "F.Fab")
 			(effects
@@
 	)
 	(segment
-		(start 36 103.16)
-		(end 36 65)
+		(start 35.499 83.978055)
+		(end 35.499 74.991946)
+		(width 2)
+		(layer "B.Cu")
+		(net 6)
+	)
+	(segment
+		(start 36.5 84.979055)
+		(end 35.499 83.978055)
 		(width 2)
 		(layer "B.Cu")
@@
 	)
 	(segment
-		(start 36 65)
+		(start 38.92 106.08)
+		(end 36.5 103.66)
+		(width 2)
+		(layer "B.Cu")
+		(net 6)
+	)
+	(segment
+		(start 36.5 64.5)
 		(end 37.265 63.735)
 		(width 2)
@@
 	)
 	(segment
-		(start 38.92 106.08)
-		(end 36 103.16)
+		(start 36.5 73.990945)
+		(end 36.5 64.5)
+		(width 2)
+		(layer "B.Cu")
+		(net 6)
+	)
+	(segment
+		(start 36.5 103.66)
+		(end 36.5 84.979055)
+		(width 2)
+		(layer "B.Cu")
+		(net 6)
+	)
+	(segment
+		(start 35.499 74.991946)
+		(end 36.5 73.990945)
 		(width 2)
 		(layer "B.Cu")
@@
 	)
 	(segment
-		(start 42 91.5)
-		(end 50 99.5)
+		(start 49.501 105.20232)
+		(end 49.501 98.736)
 		(width 2)
 		(layer "B.Cu")
@@
 	)
 	(segment
-		(start 50 99.5)
-		(end 50 105)
+		(start 49.501 98.736)
+		(end 42 91.235)
 		(width 2)
 		(layer "B.Cu")
@@
 	)
 	(segment
-		(start 53 108)
-		(end 54.42 108)
+		(start 47.735 77.735)
+		(end 52.5375 82.5375)
 		(width 2)
 		(layer "B.Cu")
@@
 	)
 	(segment
-		(start 50 105)
-		(end 53 108)
+		(start 52.29868 108)
+		(end 49.501 105.20232)
 		(width 2)
 		(layer "B.Cu")
@@
 	)
 	(segment
-		(start 53.285 84.25)
-		(end 53.25 84.25)
+		(start 52.5375 82.5375)
+		(end 54.9975 82.5375)
 		(width 2)
 		(layer "B.Cu")
@@
 	)
 	(segment
-		(start 59 90)
-		(end 53.25 84.25)
+		(start 42 77.735)
+		(end 47.735 77.735)
 		(width 2)
 		(layer "B.Cu")
@@
 	)
 	(segment
-		(start 42 91.235)
-		(end 42 91.5)
+		(start 57.921 85.461)
+		(end 57.921 106.501)
 		(width 2)
 		(layer "B.Cu")
@@
 	)
 	(segment
-		(start 55.5 108)
-		(end 59 104.5)
+		(start 57.921 106.501)
+		(end 56.422 108)
 		(width 2)
 		(layer "B.Cu")
@@
 	)
 	(segment
-		(start 54.42 108)
-		(end 55.5 108)
-		(width 2)
-		(layer "B.Cu")
-		(net 25)
-	)
-	(segment
-		(start 54.9975 82.5375)
-		(end 53.285 84.25)
-		(width 2)
-		(layer "B.Cu")
-		(net 25)
-	)
-	(segment
-		(start 53.25 84.25)
-		(end 46.735 77.735)
+		(start 56.422 108)
+		(end 54.42 108)
 		(width 2)
 		(layer "B.Cu")
@@
 	)
 	(segment
-		(start 46.735 77.735)
-		(end 42 77.735)
+		(start 54.42 108)
+		(end 52.29868 108)
 		(width 2)
 		(layer "B.Cu")
@@
 	)
 	(segment
-		(start 59 104.5)
-		(end 59 90)
+		(start 54.9975 82.5375)
+		(end 57.921 85.461)
 		(width 2)
 		(layer "B.Cu")
@@
 	)
 	(segment
-		(start 54.42 91.42)
-		(end 49.235 86.235)
-		(width 2)
-		(layer "B.Cu")
-		(net 26)
-	)
-	(segment
-		(start 54.42 103)
-		(end 54.42 91.42)
+		(start 42 72.735)
+		(end 50.146162 72.735)
 		(width 2)
 		(layer "B.Cu")
@@
 	)
 	(segment
-		(start 39 74.5)
-		(end 39 83.235)
+		(start 38.5 82.735)
+		(end 42 86.235)
 		(width 2)
 		(layer "B.Cu")
@@
 	(segment
 		(start 42 72.735)
-		(end 40.765 72.735)
+		(end 50.195 72.735)
 		(width 2)
 		(layer "B.Cu")
@@
 	)
 	(segment
-		(start 49.235 86.235)
-		(end 42 86.235)
+		(start 42 72.735)
+		(end 38.5 76.235)
 		(width 2)
 		(layer "B.Cu")
@@
 	)
 	(segment
-		(start 39 83.235)
-		(end 42 86.235)
+		(start 38.5 76.235)
+		(end 38.5 82.735)
 		(width 2)
 		(layer "B.Cu")
@@
 	)
 	(segment
-		(start 40.765 72.735)
-		(end 39 74.5)
+		(start 42 86.235)
+		(end 54.42 98.655)
 		(width 2)
 		(layer "B.Cu")
@@
 	)
 	(segment
-		(start 42 72.735)
-		(end 50.195 72.735)
+		(start 54.42 98.655)
+		(end 54.42 103)
 		(width 2)
 		(layer "B.Cu")
